File: imulogger/imulogger.sch (KiCad schematic (older format))
At the start: 26 parts, among them J1 DEBUG, J3 PWRCONN, J4 Micro_SD_Card, U1 ESP32-WROOM-32, U2 USFS, U3 AMS1117-3.3

Commit message: Revert "experiment"
This reverts commit 6fe68751296b879cc60505c4876b2cc8c070c93c.
Parts:
- added J2: USB_B_Micro, Connector_USB:USB_Micro-B_Molex-105017-0001, symbol Connector:USB_B_Micro
- added R2, R3: 220, Resistor_SMD:R_0402_1005Metric, symbol Device:R
- added R6: 0, Resistor_SMD:R_0402_1005Metric, symbol Device:R
- added SW1: EN, Button_Switch_SMD:SW_SPST_B3U-1000P, symbol Switch:SW_Push
- added SW2: BOOT, Button_Switch_SMD:SW_SPST_B3U-1000P, symbol Switch:SW_Push
- C5: symbol Device:C_Small -> Device:C
- U1: symbol imulogger-symbols:ESP32-WROOM-32 -> RF_Module:ESP32-WROOM-32
Connections:
- net EN: now also R2.2
- net GND: now also J3.2 (Pin_2), J2.5 (GND), R6.2, SW1.2, SW2.2; no longer J3.1 (Pin_1), U1.39 (THERMAL)
- net IO0: now also R3.2
- net at D1.2 (A): now also J3.1 (Pin_1), J2.1 (VBUS); no longer J3.2 (Pin_2)
- new net: R2.1, SW1.1
- new net: R3.1, SW2.1
- new net: J2.6 (Shield), R6.1
Other:
- note added: "UI"
- moved on the sheet: C5, D1, J3
Changed lines of the file:
@@
 EESchema Schematic File Version 4
-LIBS:imulogger-cache
 EELAYER 29 0
 EELAYER END
@@
 $EndDescr
 $Comp
-L imulogger-symbols:ESP32-WROOM-32 U1
+L RF_Module:ESP32-WROOM-32 U1
 U 1 1 5CB6CF70
 P 2200 3150
@@
 Text GLabel 1200 2900 3    50   Input ~ 0
 IO0
+$Comp
+L Switch:SW_Push SW1
+U 1 1 5CB8F3F3
+P 1400 7000
+F 0 "SW1" H 1400 7285 50  0000 C CNN
+F 1 "EN" H 1400 7194 50  0000 C CNN
+F 2 "Button_Switch_SMD:SW_SPST_B3U-1000P" H 1400 7200 50  0001 C CNN
+F 3 "~" H 1400 7200 50  0001 C CNN
+	1    1400 7000
+	1    0    0    -1
+$EndComp
+$Comp
+L Switch:SW_Push SW2
+U 1 1 5CB900CF
+P 1400 7400
+F 0 "SW2" H 1400 7685 50  0000 C CNN
+F 1 "BOOT" H 1400 7594 50  0000 C CNN
+F 2 "Button_Switch_SMD:SW_SPST_B3U-1000P" H 1400 7600 50  0001 C CNN
+F 3 "~" H 1400 7600 50  0001 C CNN
+	1    1400 7400
+	1    0    0    -1
+$EndComp
+$Comp
+L power:GND #PWR0109
+U 1 1 5CB90A3A
+P 1600 7000
+F 0 "#PWR0109" H 1600 6750 50  0001 C CNN
+F 1 "GND" V 1605 6872 50  0000 R CNN
+F 2 "" H 1600 7000 50  0001 C CNN
+F 3 "" H 1600 7000 50  0001 C CNN
+	1    1600 7000
+	0    -1   -1   0
+$EndComp
+$Comp
+L power:GND #PWR0110
+U 1 1 5CB913E8
+P 1600 7400
+F 0 "#PWR0110" H 1600 7150 50  0001 C CNN
+F 1 "GND" V 1605 7272 50  0000 R CNN
+F 2 "" H 1600 7400 50  0001 C CNN
+F 3 "" H 1600 7400 50  0001 C CNN
+	1    1600 7400
+	0    -1   -1   0
+$EndComp
+Text GLabel 900  7000 0    50   Input ~ 0
+EN
+Text GLabel 900  7400 0    50   Input ~ 0
+IO0
 Text Notes 1700 1150 0    315  ~ 63
 MCU
+Text Notes 1100 6350 0    315  ~ 63
+UI
 Text Notes 9350 4550 0    315  ~ 63
 uSD
@@
 Text Notes 2350 6350 0    315  ~ 63
 Prog.
+$Comp
+L Device:R R2
+U 1 1 5CBAECFB
+P 1050 7000
+F 0 "R2" V 843 7000 50  0000 C CNN
+F 1 "220" V 934 7000 50  0000 C CNN
+F 2 "Resistor_SMD:R_0402_1005Metric" V 980 7000 50  0001 C CNN
+F 3 "~" H 1050 7000 50  0001 C CNN
+	1    1050 7000
+	0    1    1    0
+$EndComp
+$Comp
+L Device:R R3
+U 1 1 5CBAF6D9
+P 1050 7400
+F 0 "R3" V 843 7400 50  0000 C CNN
+F 1 "220" V 934 7400 50  0000 C CNN
+F 2 "Resistor_SMD:R_0402_1005Metric" V 980 7400 50  0001 C CNN
+F 3 "~" H 1050 7400 50  0001 C CNN
+	1    1050 7400
+	0    1    1    0
+$EndComp
 $Comp
 L Regulator_Linear:AMS1117-3.3 U3
@@
 Power
 $Comp
+L Connector:USB_B_Micro J2
+U 1 1 5CBC3B10
+P 4900 4700
+F 0 "J2" H 4957 5167 50  0000 C CNN
+F 1 "USB_B_Micro" H 4957 5076 50  0000 C CNN
+F 2 "Connector_USB:USB_Micro-B_Molex-105017-0001" H 5050 4650 50  0001 C CNN
+F 3 "~" H 5050 4650 50  0001 C CNN
+	1    4900 4700
+	1    0    0    -1
+$EndComp
+$Comp
 L power:GND #PWR0114
 U 1 1 5CBC57D2
-P 5300 4600
-F 0 "#PWR0114" H 5300 4350 50  0001 C CNN
-F 1 "GND" H 5305 4427 50  0000 C CNN
-F 2 "" H 5300 4600 50  0001 C CNN
-F 3 "" H 5300 4600 50  0001 C CNN
-	1    5300 4600
-	1    0    0    -1
-$EndComp
+P 4900 5550
+F 0 "#PWR0114" H 4900 5300 50  0001 C CNN
+F 1 "GND" H 4905 5377 50  0000 C CNN
+F 2 "" H 4900 5550 50  0001 C CNN
+F 3 "" H 4900 5550 50  0001 C CNN
+	1    4900 5550
+	1    0    0    -1
+$EndComp
+$Comp
+L Device:R R6
+U 1 1 5CBC6039
+P 4800 5250
+F 0 "R6" H 4600 5300 50  0000 L CNN
+F 1 "0" H 4600 5200 50  0000 L CNN
+F 2 "Resistor_SMD:R_0402_1005Metric" V 4730 5250 50  0001 C CNN
+F 3 "~" H 4800 5250 50  0001 C CNN
+	1    4800 5250
+	1    0    0    -1
+$EndComp
+Wire Wire Line
+	4800 5400 4800 5450
+Wire Wire Line
+	4900 5100 4900 5450
 $Comp
 L power:+5V #PWR0115
 U 1 1 5CBC8BE3
-P 5300 4500
-F 0 "#PWR0115" H 5300 4350 50  0001 C CNN
-F 1 "+5V" H 5315 4673 50  0000 C CNN
-F 2 "" H 5300 4500 50  0001 C CNN
-F 3 "" H 5300 4500 50  0001 C CNN
-	1    5300 4500
+P 5900 4500
+F 0 "#PWR0115" H 5900 4350 50  0001 C CNN
+F 1 "+5V" H 5915 4673 50  0000 C CNN
+F 2 "" H 5900 4500 50  0001 C CNN
+F 3 "" H 5900 4500 50  0001 C CNN
+	1    5900 4500
 	1    0    0    -1
 $EndComp
@@
 L Device:D D1
 U 1 1 5CBCA271
-P 4950 4500
-F 0 "D1" H 4950 4284 50  0000 C CNN
-F 1 "BAS3010" H 4950 4375 50  0000 C CNN
-F 2 "Diode_SMD:D_SOD-323" H 4950 4500 50  0001 C CNN
-F 3 "~" H 4950 4500 50  0001 C CNN
-	1    4950 4500
+P 5650 4500
+F 0 "D1" H 5650 4284 50  0000 C CNN
+F 1 "BAS3010" H 5650 4375 50  0000 C CNN
+F 2 "Diode_SMD:D_SOD-323" H 5650 4500 50  0001 C CNN
+F 3 "~" H 5650 4500 50  0001 C CNN
+	1    5650 4500
 	-1   0    0    1
 $EndComp
 $Comp
-L Device:C_Small C5
+L Device:C C5
 U 1 1 5CBCC768
-P 5600 4550
-F 0 "C5" H 5715 4596 50  0000 L CNN
-F 1 "100n" H 5715 4505 50  0000 L CNN
-F 2 "Capacitor_SMD:C_0402_1005Metric" H 5638 4400 50  0001 C CNN
-F 3 "~" H 5600 4550 50  0001 C CNN
-	1    5600 4550
+P 5900 4750
+F 0 "C5" H 6015 4796 50  0000 L CNN
+F 1 "100n" H 6015 4705 50  0000 L CNN
+F 2 "Capacitor_SMD:C_0402_1005Metric" H 5938 4600 50  0001 C CNN
+F 3 "~" H 5900 4750 50  0001 C CNN
+	1    5900 4750
+	1    0    0    -1
+$EndComp
+Wire Wire Line
+	5800 4500 5900 4500
+Wire Wire Line
+	5900 4500 5900 4600
+Connection ~ 5900 4500
+$Comp
+L power:GND #PWR0116
+U 1 1 5CBCE0A5
+P 5900 4900
+F 0 "#PWR0116" H 5900 4650 50  0001 C CNN
+F 1 "GND" H 5905 4727 50  0000 C CNN
+F 2 "" H 5900 4900 50  0001 C CNN
+F 3 "" H 5900 4900 50  0001 C CNN
+	1    5900 4900
 	1    0    0    -1
 $EndComp
@@
 L Connector_Generic:Conn_01x02 J3
 U 1 1 5CBD250B
-P 4600 4600
-F 0 "J3" H 4680 4592 50  0000 L CNN
-F 1 "PWRCONN" H 4680 4501 50  0000 L CNN
-F 2 "Connector_PinHeader_2.54mm:PinHeader_1x02_P2.54mm_Horizontal" H 4600 4600 50  0001 C CNN
-F 3 "~" H 4600 4600 50  0001 C CNN
-	1    4600 4600
-	-1   0    0    1
-$EndComp
+P 5550 5350
+F 0 "J3" H 5630 5342 50  0000 L CNN
+F 1 "PWRCONN" H 5630 5251 50  0000 L CNN
+F 2 "Connector_PinHeader_2.54mm:PinHeader_1x02_P2.54mm_Horizontal" H 5550 5350 50  0001 C CNN
+F 3 "~" H 5550 5350 50  0001 C CNN
+	1    5550 5350
+	1    0    0    -1
+$EndComp
+Wire Wire Line
+	5200 4500 5350 4500
+Wire Wire Line
+	5350 5450 4900 5450
+Connection ~ 4900 5450
+Wire Wire Line
+	5350 5350 5350 4500
+Connection ~ 5350 4500
+Wire Wire Line
+	5350 4500 5500 4500
 Text Notes 4750 4000 0    315  ~ 63
 USB
@@
 Wire Wire Line
 	2900 7200 2600 7200
-$Comp
-L power:GND #PWR0117
-U 1 1 5CB7F7EB
-P 2350 4550
-F 0 "#PWR0117" H 2350 4300 50  0001 C CNN
-F 1 "GND" H 2355 4377 50  0000 C CNN
-F 2 "" H 2350 4550 50  0001 C CNN
-F 3 "" H 2350 4550 50  0001 C CNN
-	1    2350 4550
-	1    0    0    -1
-$EndComp
-Wire Wire Line
-	5300 4500 5100 4500
-Wire Wire Line
-	4800 4600 5300 4600
-Wire Wire Line
-	5450 4650 5450 4600
-Wire Wire Line
-	5450 4600 5300 4600
-Connection ~ 5300 4600
-Wire Wire Line
-	5600 4450 5450 4450
-Wire Wire Line
-	5450 4450 5450 4500
-Wire Wire Line
-	5450 4500 5300 4500
-Connection ~ 5300 4500
-Wire Wire Line
-	5450 4650 5600 4650
+Wire Wire Line
+	4800 5450 4900 5450
+Wire Wire Line
+	4900 5450 4900 5550
 $EndSCHEMATC

Commit message: experiment
Parts:
- removed J2: USB_B_Micro, Connector_USB:USB_Micro-B_Molex-105017-0001, symbol Connector:USB_B_Micro
- removed R2, R3: 220, Resistor_SMD:R_0402_1005Metric, symbol Device:R
- removed R6: 0, Resistor_SMD:R_0402_1005Metric, symbol Device:R
- removed SW1: EN, Button_Switch_SMD:SW_SPST_B3U-1000P, symbol Switch:SW_Push
- removed SW2: BOOT, Button_Switch_SMD:SW_SPST_B3U-1000P, symbol Switch:SW_Push
- C5: symbol Device:C -> Device:C_Small
- U1: symbol RF_Module:ESP32-WROOM-32 -> imulogger-symbols:ESP32-WROOM-32
Connections:
- net GND: now also J3.1 (Pin_1), U1.39 (THERMAL); no longer J3.2 (Pin_2)
- net at D1.2 (A): now also J3.2 (Pin_2); no longer J3.1 (Pin_1)
Other:
- note removed: "UI"
- moved on the sheet: C5, D1, J3
Changed lines of the file:
@@
 EESchema Schematic File Version 4
+LIBS:imulogger-cache
 EELAYER 29 0
 EELAYER END
@@
 $EndDescr
 $Comp
-L RF_Module:ESP32-WROOM-32 U1
+L imulogger-symbols:ESP32-WROOM-32 U1
 U 1 1 5CB6CF70
 P 2200 3150
@@
 Text GLabel 1200 2900 3    50   Input ~ 0
 IO0
-$Comp
-L Switch:SW_Push SW1
-U 1 1 5CB8F3F3
-P 1400 7000
-F 0 "SW1" H 1400 7285 50  0000 C CNN
-F 1 "EN" H 1400 7194 50  0000 C CNN
-F 2 "Button_Switch_SMD:SW_SPST_B3U-1000P" H 1400 7200 50  0001 C CNN
-F 3 "~" H 1400 7200 50  0001 C CNN
-	1    1400 7000
-	1    0    0    -1
-$EndComp
-$Comp
-L Switch:SW_Push SW2
-U 1 1 5CB900CF
-P 1400 7400
-F 0 "SW2" H 1400 7685 50  0000 C CNN
-F 1 "BOOT" H 1400 7594 50  0000 C CNN
-F 2 "Button_Switch_SMD:SW_SPST_B3U-1000P" H 1400 7600 50  0001 C CNN
-F 3 "~" H 1400 7600 50  0001 C CNN
-	1    1400 7400
-	1    0    0    -1
-$EndComp
-$Comp
-L power:GND #PWR0109
-U 1 1 5CB90A3A
-P 1600 7000
-F 0 "#PWR0109" H 1600 6750 50  0001 C CNN
-F 1 "GND" V 1605 6872 50  0000 R CNN
-F 2 "" H 1600 7000 50  0001 C CNN
-F 3 "" H 1600 7000 50  0001 C CNN
-	1    1600 7000
-	0    -1   -1   0
-$EndComp
-$Comp
-L power:GND #PWR0110
-U 1 1 5CB913E8
-P 1600 7400
-F 0 "#PWR0110" H 1600 7150 50  0001 C CNN
-F 1 "GND" V 1605 7272 50  0000 R CNN
-F 2 "" H 1600 7400 50  0001 C CNN
-F 3 "" H 1600 7400 50  0001 C CNN
-	1    1600 7400
-	0    -1   -1   0
-$EndComp
-Text GLabel 900  7000 0    50   Input ~ 0
-EN
-Text GLabel 900  7400 0    50   Input ~ 0
-IO0
 Text Notes 1700 1150 0    315  ~ 63
 MCU
-Text Notes 1100 6350 0    315  ~ 63
-UI
 Text Notes 9350 4550 0    315  ~ 63
 uSD
@@
 Text Notes 2350 6350 0    315  ~ 63
 Prog.
-$Comp
-L Device:R R2
-U 1 1 5CBAECFB
-P 1050 7000
-F 0 "R2" V 843 7000 50  0000 C CNN
-F 1 "220" V 934 7000 50  0000 C CNN
-F 2 "Resistor_SMD:R_0402_1005Metric" V 980 7000 50  0001 C CNN
-F 3 "~" H 1050 7000 50  0001 C CNN
-	1    1050 7000
-	0    1    1    0
-$EndComp
-$Comp
-L Device:R R3
-U 1 1 5CBAF6D9
-P 1050 7400
-F 0 "R3" V 843 7400 50  0000 C CNN
-F 1 "220" V 934 7400 50  0000 C CNN
-F 2 "Resistor_SMD:R_0402_1005Metric" V 980 7400 50  0001 C CNN
-F 3 "~" H 1050 7400 50  0001 C CNN
-	1    1050 7400
-	0    1    1    0
-$EndComp
 $Comp
 L Regulator_Linear:AMS1117-3.3 U3
@@
 Power
 $Comp
-L Connector:USB_B_Micro J2
-U 1 1 5CBC3B10
-P 4900 4700
-F 0 "J2" H 4957 5167 50  0000 C CNN
-F 1 "USB_B_Micro" H 4957 5076 50  0000 C CNN
-F 2 "Connector_USB:USB_Micro-B_Molex-105017-0001" H 5050 4650 50  0001 C CNN
-F 3 "~" H 5050 4650 50  0001 C CNN
-	1    4900 4700
-	1    0    0    -1
-$EndComp
-$Comp
 L power:GND #PWR0114
 U 1 1 5CBC57D2
-P 4900 5550
-F 0 "#PWR0114" H 4900 5300 50  0001 C CNN
-F 1 "GND" H 4905 5377 50  0000 C CNN
-F 2 "" H 4900 5550 50  0001 C CNN
-F 3 "" H 4900 5550 50  0001 C CNN
-	1    4900 5550
-	1    0    0    -1
-$EndComp
-$Comp
-L Device:R R6
-U 1 1 5CBC6039
-P 4800 5250
-F 0 "R6" H 4600 5300 50  0000 L CNN
-F 1 "0" H 4600 5200 50  0000 L CNN
-F 2 "Resistor_SMD:R_0402_1005Metric" V 4730 5250 50  0001 C CNN
-F 3 "~" H 4800 5250 50  0001 C CNN
-	1    4800 5250
-	1    0    0    -1
-$EndComp
-Wire Wire Line
-	4800 5400 4800 5450
-Wire Wire Line
-	4900 5100 4900 5450
+P 5300 4600
+F 0 "#PWR0114" H 5300 4350 50  0001 C CNN
+F 1 "GND" H 5305 4427 50  0000 C CNN
+F 2 "" H 5300 4600 50  0001 C CNN
+F 3 "" H 5300 4600 50  0001 C CNN
+	1    5300 4600
+	1    0    0    -1
+$EndComp
 $Comp
 L power:+5V #PWR0115
 U 1 1 5CBC8BE3
-P 5900 4500
-F 0 "#PWR0115" H 5900 4350 50  0001 C CNN
-F 1 "+5V" H 5915 4673 50  0000 C CNN
-F 2 "" H 5900 4500 50  0001 C CNN
-F 3 "" H 5900 4500 50  0001 C CNN
-	1    5900 4500
+P 5300 4500
+F 0 "#PWR0115" H 5300 4350 50  0001 C CNN
+F 1 "+5V" H 5315 4673 50  0000 C CNN
+F 2 "" H 5300 4500 50  0001 C CNN
+F 3 "" H 5300 4500 50  0001 C CNN
+	1    5300 4500
 	1    0    0    -1
 $EndComp
@@
 L Device:D D1
 U 1 1 5CBCA271
-P 5650 4500
-F 0 "D1" H 5650 4284 50  0000 C CNN
-F 1 "BAS3010" H 5650 4375 50  0000 C CNN
-F 2 "Diode_SMD:D_SOD-323" H 5650 4500 50  0001 C CNN
-F 3 "~" H 5650 4500 50  0001 C CNN
-	1    5650 4500
+P 4950 4500
+F 0 "D1" H 4950 4284 50  0000 C CNN
+F 1 "BAS3010" H 4950 4375 50  0000 C CNN
+F 2 "Diode_SMD:D_SOD-323" H 4950 4500 50  0001 C CNN
+F 3 "~" H 4950 4500 50  0001 C CNN
+	1    4950 4500
 	-1   0    0    1
 $EndComp
 $Comp
-L Device:C C5
+L Device:C_Small C5
 U 1 1 5CBCC768
-P 5900 4750
-F 0 "C5" H 6015 4796 50  0000 L CNN
-F 1 "100n" H 6015 4705 50  0000 L CNN
-F 2 "Capacitor_SMD:C_0402_1005Metric" H 5938 4600 50  0001 C CNN
-F 3 "~" H 5900 4750 50  0001 C CNN
-	1    5900 4750
-	1    0    0    -1
-$EndComp
-Wire Wire Line
-	5800 4500 5900 4500
-Wire Wire Line
-	5900 4500 5900 4600
-Connection ~ 5900 4500
-$Comp
-L power:GND #PWR0116
-U 1 1 5CBCE0A5
-P 5900 4900
-F 0 "#PWR0116" H 5900 4650 50  0001 C CNN
-F 1 "GND" H 5905 4727 50  0000 C CNN
-F 2 "" H 5900 4900 50  0001 C CNN
-F 3 "" H 5900 4900 50  0001 C CNN
-	1    5900 4900
+P 5600 4550
+F 0 "C5" H 5715 4596 50  0000 L CNN
+F 1 "100n" H 5715 4505 50  0000 L CNN
+F 2 "Capacitor_SMD:C_0402_1005Metric" H 5638 4400 50  0001 C CNN
+F 3 "~" H 5600 4550 50  0001 C CNN
+	1    5600 4550
 	1    0    0    -1
 $EndComp
@@
 L Connector_Generic:Conn_01x02 J3
 U 1 1 5CBD250B
-P 5550 5350
-F 0 "J3" H 5630 5342 50  0000 L CNN
-F 1 "PWRCONN" H 5630 5251 50  0000 L CNN
-F 2 "Connector_PinHeader_2.54mm:PinHeader_1x02_P2.54mm_Horizontal" H 5550 5350 50  0001 C CNN
-F 3 "~" H 5550 5350 50  0001 C CNN
-	1    5550 5350
-	1    0    0    -1
-$EndComp
-Wire Wire Line
-	5200 4500 5350 4500
-Wire Wire Line
-	5350 5450 4900 5450
-Connection ~ 4900 5450
-Wire Wire Line
-	5350 5350 5350 4500
-Connection ~ 5350 4500
-Wire Wire Line
-	5350 4500 5500 4500
+P 4600 4600
+F 0 "J3" H 4680 4592 50  0000 L CNN
+F 1 "PWRCONN" H 4680 4501 50  0000 L CNN
+F 2 "Connector_PinHeader_2.54mm:PinHeader_1x02_P2.54mm_Horizontal" H 4600 4600 50  0001 C CNN
+F 3 "~" H 4600 4600 50  0001 C CNN
+	1    4600 4600
+	-1   0    0    1
+$EndComp
 Text Notes 4750 4000 0    315  ~ 63
 USB
@@
 Wire Wire Line
 	2900 7200 2600 7200
-Wire Wire Line
-	4800 5450 4900 5450
-Wire Wire Line
-	4900 5450 4900 5550
+$Comp
+L power:GND #PWR0117
+U 1 1 5CB7F7EB
+P 2350 4550
+F 0 "#PWR0117" H 2350 4300 50  0001 C CNN
+F 1 "GND" H 2355 4377 50  0000 C CNN
+F 2 "" H 2350 4550 50  0001 C CNN
+F 3 "" H 2350 4550 50  0001 C CNN
+	1    2350 4550
+	1    0    0    -1
+$EndComp
+Wire Wire Line
+	5300 4500 5100 4500
+Wire Wire Line
+	4800 4600 5300 4600
+Wire Wire Line
+	5450 4650 5450 4600
+Wire Wire Line
+	5450 4600 5300 4600
+Connection ~ 5300 4600
+Wire Wire Line
+	5600 4450 5450 4450
+Wire Wire Line
+	5450 4450 5450 4500
+Wire Wire Line
+	5450 4500 5300 4500
+Connection ~ 5300 4500
+Wire Wire Line
+	5450 4650 5600 4650
 $EndSCHEMATC
