File: imulogger/imulogger.sch (KiCad schematic (older format))
At the start: 24 parts, among them J1 DEBUG, J3 PWRCONN, J4 Micro_SD_Card, U1 ESP32-WROOM-32, U2 USFS, U3 AMS1117-3.3

Commit message: imulogger: use our custom esp32 footprint
Parts:
- U1: footprint RF_Module:ESP32-WROOM-32 -> imulogger-footprints:ESP32-WROOM-32
Changed lines of the file:
@@
 F 0 "U1" H 2200 4850 50  0000 C CNN
 F 1 "ESP32-WROOM-32" H 2200 4750 50  0000 C CNN
-F 2 "RF_Module:ESP32-WROOM-32" H 2200 1650 50  0001 C CNN
+F 2 "imulogger-footprints:ESP32-WROOM-32" H 2200 1650 50  0001 C CNN
 F 3 "https://www.espressif.com/sites/default/files/documentation/esp32-wroom-32_datasheet_en.pdf" H 1900 3200 50  0001 C CNN
 	1    2200 3150

Commit message: redesign power supply
- add battery and charger
- use LDO with a proper dropout voltage
Parts:
- removed C5: 100n, Capacitor_SMD:C_0402_1005Metric, symbol Device:C
- removed D1: BAS3010, Diode_SMD:D_SOD-323, symbol Device:D
- removed J3: PWRCONN, Connector_PinHeader_2.54mm:PinHeader_1x02_P2.54mm_Horizontal, symbol Connector_Generic:Conn_01x02
- added C10, C9: 4.7u, symbol Device:C_Small
- added D2: LED, symbol Device:LED
- added D3, D4: BAT20J, symbol Device:D_Schottky
- added J2: BATCONN, Connector_PinHeader_2.54mm:PinHeader_1x02_P2.54mm_Horizontal, symbol Connector_Generic:Conn_01x02
- added J5: PWRCONN, Connector_PinHeader_2.54mm:PinHeader_1x02_P2.54mm_Horizontal, symbol Connector_Generic:Conn_01x02
- added Q1: TP0610T, Package_TO_SOT_SMD:SOT-23, symbol Transistor_FET:TP0610T
- added R2: nc, Resistor_SMD:R_0402_1005Metric, symbol Device:R_Small
- added R3: 2k, symbol Device:R_Small
- added R6: 470, symbol Device:R_Small
- added R8: 10k, symbol Device:R_Small
- added U4: MCP73831-2-OT, Package_TO_SOT_SMD:SOT-23-5, symbol Battery_Management:MCP73831-2-OT
- U3: value AMS1117-3.3 -> MCP1826S; symbol Regulator_Linear:AMS1117-3.3 -> Regulator_Linear:MCP1826S
Connections:
- net labels added: V_BAT, V_EXT
- net labels removed: +5V
- wire segments 66 -> 110
Other:
- note added: "Bat + Charger"
- note added: "PwrSrcSel + Reg"
- note removed: "Power"
- note removed: "USB"
- moved on the sheet: C3, C4, C6, J1, R5

Commit message: Revert "imulogger: use 47K pull-ups for sdcard"
This reverts commit df5adce347d57e44a57313ac28780a91eea5d007.

10K is the value recommended by espressif and it's closer to olimex' 2.2k
Parts:
- R11, R13, R14, R7, R9: value 47K -> 10K
Changed lines of the file:
@@
 P 8950 4950
 F 0 "R14" H 9000 5000 50  0000 L CNN
-F 1 "47K" H 9000 4900 50  0000 L CNN
+F 1 "10K" H 9000 4900 50  0000 L CNN
 F 2 "Resistor_SMD:R_0402_1005Metric" H 8950 4950 50  0001 C CNN
 F 3 "~" H 8950 4950 50  0001 C CNN
@@
 P 8850 4650
 F 0 "R13" H 8900 4700 50  0000 L CNN
-F 1 "47K" H 8900 4600 50  0000 L CNN
+F 1 "10K" H 8900 4600 50  0000 L CNN
 F 2 "Resistor_SMD:R_0402_1005Metric" H 8850 4650 50  0001 C CNN
 F 3 "~" H 8850 4650 50  0001 C CNN
@@
 P 8400 4950
 F 0 "R7" H 8450 5000 50  0000 L CNN
-F 1 "47K" H 8450 4900 50  0000 L CNN
+F 1 "10K" H 8450 4900 50  0000 L CNN
 F 2 "Resistor_SMD:R_0402_1005Metric" H 8400 4950 50  0001 C CNN
 F 3 "~" H 8400 4950 50  0001 C CNN
@@
 P 8550 4650
 F 0 "R9" H 8600 4700 50  0000 L CNN
-F 1 "47K" H 8600 4600 50  0000 L CNN
+F 1 "10K" H 8600 4600 50  0000 L CNN
 F 2 "Resistor_SMD:R_0402_1005Metric" H 8550 4650 50  0001 C CNN
 F 3 "~" H 8550 4650 50  0001 C CNN
@@
 P 8650 4950
 F 0 "R11" H 8700 5000 50  0000 L CNN
-F 1 "47K" H 8700 4900 50  0000 L CNN
+F 1 "10K" H 8700 4900 50  0000 L CNN
 F 2 "Resistor_SMD:R_0402_1005Metric" H 8650 4950 50  0001 C CNN
 F 3 "~" H 8650 4950 50  0001 C CNN

Commit message: imulogger: assign footprints
Parts:
- C10, C9: footprint (none) -> Capacitor_SMD:C_0402_1005Metric
- D2: footprint (none) -> LED_SMD:LED_0402_1005Metric
- D3, D4: footprint (none) -> Diode_SMD:D_SOD-323
- J2, J5: footprint Connector_PinHeader_2.54mm:PinHeader_1x02_P2.54mm_Horizontal -> Connector_JST:JST_PH_S2B-PH-SM4-TB_1x02-1MP_P2.00mm_Horizontal
- R3, R6, R8: footprint (none) -> Resistor_SMD:R_0402_1005Metric
- U3: footprint Package_TO_SOT_SMD:SOT-223 -> imulogger-footprints:SOT-223; symbol Regulator_Linear:MCP1826S -> imulogger-symbols:MCP1826S
Changed lines of the file:
@@
 F 0 "C9" H 4592 1946 50  0000 L CNN
 F 1 "4.7u" H 4592 1855 50  0000 L CNN
-F 2 "" H 4500 1900 50  0001 C CNN
+F 2 "Capacitor_SMD:C_0402_1005Metric" H 4500 1900 50  0001 C CNN
 F 3 "~" H 4500 1900 50  0001 C CNN
 	1    4500 1900
@@
 F 0 "C10" H 6142 1896 50  0000 L CNN
 F 1 "4.7u" H 6142 1805 50  0000 L CNN
-F 2 "" H 6050 1850 50  0001 C CNN
+F 2 "Capacitor_SMD:C_0402_1005Metric" H 6050 1850 50  0001 C CNN
 F 3 "~" H 6050 1850 50  0001 C CNN
 	1    6050 1850
@@
 F 0 "R3" H 5009 2196 50  0000 L CNN
 F 1 "2k" H 5009 2105 50  0000 L CNN
-F 2 "" H 4950 2150 50  0001 C CNN
+F 2 "Resistor_SMD:R_0402_1005Metric" H 4950 2150 50  0001 C CNN
 F 3 "~" H 4950 2150 50  0001 C CNN
 	1    4950 2150
@@
 F 0 "D2" V 6689 1783 50  0000 R CNN
 F 1 "LED" V 6598 1783 50  0000 R CNN
-F 2 "" H 6650 1900 50  0001 C CNN
+F 2 "LED_SMD:LED_0402_1005Metric" H 6650 1900 50  0001 C CNN
 F 3 "~" H 6650 1900 50  0001 C CNN
 	1    6650 1900
@@
 F 0 "R6" V 6354 2050 50  0000 C CNN
 F 1 "470" V 6445 2050 50  0000 C CNN
-F 2 "" H 6550 2050 50  0001 C CNN
+F 2 "Resistor_SMD:R_0402_1005Metric" H 6550 2050 50  0001 C CNN
 F 3 "~" H 6550 2050 50  0001 C CNN
 	1    6550 2050
@@
 F 0 "J2" H 4580 2692 50  0000 L CNN
 F 1 "BATCONN" H 4580 2601 50  0000 L CNN
-F 2 "Connector_PinHeader_2.54mm:PinHeader_1x02_P2.54mm_Horizontal" H 4500 2700 50  0001 C CNN
+F 2 "Connector_JST:JST_PH_S2B-PH-SM4-TB_1x02-1MP_P2.00mm_Horizontal" H 4500 2700 50  0001 C CNN
 F 3 "~" H 4500 2700 50  0001 C CNN
 	1    4500 2700
@@
 F 0 "D4" H 2200 7184 50  0000 C CNN
 F 1 "BAT20J" H 2200 7275 50  0000 C CNN
-F 2 "" H 2200 7400 50  0001 C CNN
+F 2 "Diode_SMD:D_SOD-323" H 2200 7400 50  0001 C CNN
 F 3 "~" H 2200 7400 50  0001 C CNN
 	1    2200 7400
@@
 F 0 "R8" H 1709 7196 50  0000 L CNN
 F 1 "10k" H 1709 7105 50  0000 L CNN
-F 2 "" H 1650 7150 50  0001 C CNN
+F 2 "Resistor_SMD:R_0402_1005Metric" H 1650 7150 50  0001 C CNN
 F 3 "~" H 1650 7150 50  0001 C CNN
 	1    1650 7150
@@
 $EndComp
 $Comp
-L Regulator_Linear:MCP1826S U3
+L imulogger-symbols:V_EXT #PWR08
+U 1 1 5CC5AA7B
+P 1650 6700
+F 0 "#PWR08" H 1650 6550 50  0001 C CNN
+F 1 "V_EXT" H 1667 6873 50  0000 C CNN
+F 2 "" H 1650 6700 50  0001 C CNN
+F 3 "" H 1650 6700 50  0001 C CNN
+	1    1650 6700
+	1    0    0    -1
+$EndComp
+Wire Wire Line
+	1650 6700 1650 6900
+Connection ~ 1650 6900
+$Comp
+L Connector_Generic:Conn_01x02 J5
+U 1 1 5CC7E791
+P 1000 7000
+F 0 "J5" H 1080 6992 50  0000 L CNN
+F 1 "PWRCONN" H 1080 6901 50  0000 L CNN
+F 2 "Connector_JST:JST_PH_S2B-PH-SM4-TB_1x02-1MP_P2.00mm_Horizontal" H 1000 7000 50  0001 C CNN
+F 3 "~" H 1000 7000 50  0001 C CNN
+	1    1000 7000
+	-1   0    0    1
+$EndComp
+$Comp
+L Device:D_Schottky D3
+U 1 1 5CC86772
+P 1450 6900
+F 0 "D3" H 1450 6684 50  0000 C CNN
+F 1 "BAT20J" H 1450 6775 50  0000 C CNN
+F 2 "Diode_SMD:D_SOD-323" H 1450 6900 50  0001 C CNN
+F 3 "~" H 1450 6900 50  0001 C CNN
+	1    1450 6900
+	-1   0    0    1
+$EndComp
+Wire Wire Line
+	1200 7000 1200 7300
+Wire Wire Line
+	1200 7300 1650 7300
+Wire Wire Line
+	1650 7300 1650 7250
+Wire Wire Line
+	1650 7350 1650 7300
+Connection ~ 1650 7300
+Wire Wire Line
+	2450 7400 3050 7400
+Wire Wire Line
+	3050 7400 3050 6950
+Wire Wire Line
+	3050 6950 3450 6950
+Connection ~ 2450 7400
+$Comp
+L imulogger-symbols:V_BAT #PWR06
+U 1 1 5CCA121B
+P 4800 2700
+F 0 "#PWR06" H 4800 2550 50  0001 C CNN
+F 1 "V_BAT" H 4818 2873 50  0000 C CNN
+F 2 "" H 4800 2700 50  0001 C CNN
+F 3 "" H 4800 2700 50  0001 C CNN
+	1    4800 2700
+	-1   0    0    1
+$EndComp
+Connection ~ 4800 2700
+$Comp
+L imulogger-symbols:V_EXT #PWR011
+U 1 1 5CCAA8B1
+P 5450 1450
+F 0 "#PWR011" H 5450 1300 50  0001 C CNN
+F 1 "V_EXT" H 5467 1623 50  0000 C CNN
+F 2 "" H 5450 1450 50  0001 C CNN
+F 3 "" H 5450 1450 50  0001 C CNN
+	1    5450 1450
+	1    0    0    -1
+$EndComp
+$Comp
+L power:PWR_FLAG #FLG0101
+U 1 1 5CCBA902
+P 1200 7300
+F 0 "#FLG0101" H 1200 7375 50  0001 C CNN
+F 1 "PWR_FLAG" H 1200 7473 50  0000 C CNN
+F 2 "" H 1200 7300 50  0001 C CNN
+F 3 "~" H 1200 7300 50  0001 C CNN
+	1    1200 7300
+	-1   0    0    1
+$EndComp
+Connection ~ 1200 7300
+$Comp
+L power:PWR_FLAG #FLG0102
+U 1 1 5CCBB45A
+P 1250 6700
+F 0 "#FLG0102" H 1250 6775 50  0001 C CNN
+F 1 "PWR_FLAG" H 1250 6873 50  0000 C CNN
+F 2 "" H 1250 6700 50  0001 C CNN
+F 3 "~" H 1250 6700 50  0001 C CNN
+	1    1250 6700
+	1    0    0    -1
+$EndComp
+Wire Wire Line
+	1600 6900 1650 6900
+Wire Wire Line
+	1200 6900 1250 6900
+Wire Wire Line
+	1250 6700 1250 6900
+Connection ~ 1250 6900
+Wire Wire Line
+	1250 6900 1300 6900
+Wire Wire Line
+	4800 2700 6350 2700
+Wire Wire Line
+	4700 2600 5200 2600
+$Comp
+L power:PWR_FLAG #FLG0103
+U 1 1 5CCCA68F
+P 3050 7400
+F 0 "#FLG0103" H 3050 7475 50  0001 C CNN
+F 1 "PWR_FLAG" H 3050 7573 50  0000 C CNN
+F 2 "" H 3050 7400 50  0001 C CNN
+F 3 "~" H 3050 7400 50  0001 C CNN
+	1    3050 7400
+	-1   0    0    1
+$EndComp
+Connection ~ 3050 7400
+$Comp
+L power:GND #PWR0110
+U 1 1 5CCF0437
+P 3900 6750
+F 0 "#PWR0110" H 3900 6500 50  0001 C CNN
+F 1 "GND" H 3905 6577 50  0000 C CNN
+F 2 "" H 3900 6750 50  0001 C CNN
+F 3 "" H 3900 6750 50  0001 C CNN
+	1    3900 6750
+	-1   0    0    1
+$EndComp
+$Comp
+L imulogger-symbols:MCP1826S U3
 U 1 1 5CBB01E6
 P 3900 6950
 F 0 "U3" H 3900 7192 50  0000 C CNN
 F 1 "MCP1826S" H 3900 7101 50  0000 C CNN
-F 2 "Package_TO_SOT_SMD:SOT-223" H 3900 7150 50  0001 C CNN
+F 2 "imulogger-footprints:SOT-223" H 3900 7150 50  0001 C CNN
 F 3 "http://www.advanced-monolithic.com/pdf/ds1117.pdf" H 4000 6700 50  0001 C CNN
 	1    3900 6950
@@
 	1    0    0    -1
 $EndComp
-$Comp
-L imulogger-symbols:V_EXT #PWR08
-U 1 1 5CC5AA7B
-P 1650 6700
-F 0 "#PWR08" H 1650 6550 50  0001 C CNN
-F 1 "V_EXT" H 1667 6873 50  0000 C CNN
-F 2 "" H 1650 6700 50  0001 C CNN
-F 3 "" H 1650 6700 50  0001 C CNN
-	1    1650 6700
-	1    0    0    -1
-$EndComp
-Wire Wire Line
-	1650 6700 1650 6900
-Connection ~ 1650 6900
-$Comp
-L Connector_Generic:Conn_01x02 J5
-U 1 1 5CC7E791
-P 1000 7000
-F 0 "J5" H 1080 6992 50  0000 L CNN
-F 1 "PWRCONN" H 1080 6901 50  0000 L CNN
-F 2 "Connector_PinHeader_2.54mm:PinHeader_1x02_P2.54mm_Horizontal" H 1000 7000 50  0001 C CNN
-F 3 "~" H 1000 7000 50  0001 C CNN
-	1    1000 7000
-	-1   0    0    1
-$EndComp
-$Comp
-L Device:D_Schottky D3
-U 1 1 5CC86772
-P 1450 6900
-F 0 "D3" H 1450 6684 50  0000 C CNN
-F 1 "BAT20J" H 1450 6775 50  0000 C CNN
-F 2 "" H 1450 6900 50  0001 C CNN
-F 3 "~" H 1450 6900 50  0001 C CNN
-	1    1450 6900
-	-1   0    0    1
-$EndComp
-Wire Wire Line
-	1200 7000 1200 7300
-Wire Wire Line
-	1200 7300 1650 7300
-Wire Wire Line
-	1650 7300 1650 7250
-Wire Wire Line
-	1650 7350 1650 7300
-Connection ~ 1650 7300
-Wire Wire Line
-	2450 7400 3050 7400
-Wire Wire Line
-	3050 7400 3050 6950
-Wire Wire Line
-	3050 6950 3450 6950
-Connection ~ 2450 7400
-$Comp
-L imulogger-symbols:V_BAT #PWR06
-U 1 1 5CCA121B
-P 4800 2700
-F 0 "#PWR06" H 4800 2550 50  0001 C CNN
-F 1 "V_BAT" H 4818 2873 50  0000 C CNN
-F 2 "" H 4800 2700 50  0001 C CNN
-F 3 "" H 4800 2700 50  0001 C CNN
-	1    4800 2700
-	-1   0    0    1
-$EndComp
-Connection ~ 4800 2700
-$Comp
-L imulogger-symbols:V_EXT #PWR011
-U 1 1 5CCAA8B1
-P 5450 1450
-F 0 "#PWR011" H 5450 1300 50  0001 C CNN
-F 1 "V_EXT" H 5467 1623 50  0000 C CNN
-F 2 "" H 5450 1450 50  0001 C CNN
-F 3 "" H 5450 1450 50  0001 C CNN
-	1    5450 1450
-	1    0    0    -1
-$EndComp
-$Comp
-L power:PWR_FLAG #FLG0101
-U 1 1 5CCBA902
-P 1200 7300
-F 0 "#FLG0101" H 1200 7375 50  0001 C CNN
-F 1 "PWR_FLAG" H 1200 7473 50  0000 C CNN
-F 2 "" H 1200 7300 50  0001 C CNN
-F 3 "~" H 1200 7300 50  0001 C CNN
-	1    1200 7300
-	-1   0    0    1
-$EndComp
-Connection ~ 1200 7300
-$Comp
-L power:PWR_FLAG #FLG0102
-U 1 1 5CCBB45A
-P 1250 6700
-F 0 "#FLG0102" H 1250 6775 50  0001 C CNN
-F 1 "PWR_FLAG" H 1250 6873 50  0000 C CNN
-F 2 "" H 1250 6700 50  0001 C CNN
-F 3 "~" H 1250 6700 50  0001 C CNN
-	1    1250 6700
-	1    0    0    -1
-$EndComp
-Wire Wire Line
-	1600 6900 1650 6900
-Wire Wire Line
-	1200 6900 1250 6900
-Wire Wire Line
-	1250 6700 1250 6900
-Connection ~ 1250 6900
-Wire Wire Line
-	1250 6900 1300 6900
-Wire Wire Line
-	4800 2700 6350 2700
-Wire Wire Line
-	4700 2600 5200 2600
-$Comp
-L power:PWR_FLAG #FLG0103
-U 1 1 5CCCA68F
-P 3050 7400
-F 0 "#FLG0103" H 3050 7475 50  0001 C CNN
-F 1 "PWR_FLAG" H 3050 7573 50  0000 C CNN
-F 2 "" H 3050 7400 50  0001 C CNN
-F 3 "~" H 3050 7400 50  0001 C CNN
-	1    3050 7400
-	-1   0    0    1
-$EndComp
-Connection ~ 3050 7400
 $EndSCHEMATC

Commit message: new pcb layout
Parts:
- removed C6: nc, Capacitor_SMD:C_0402_1005Metric, symbol Device:C
- removed R17, R5: nc, Resistor_SMD:R_0402_1005Metric, symbol Device:R_Small
- C1, C10, C2, C7, C8, C9: footprint Capacitor_SMD:C_0402_1005Metric -> Capacitor_SMD:C_0805_2012Metric_Pad1.15x1.40mm_HandSolder
- C3, C4: footprint Capacitor_SMD:C_0805_2012Metric -> Capacitor_SMD:C_0805_2012Metric_Pad1.15x1.40mm_HandSolder
- D2: footprint LED_SMD:LED_0402_1005Metric -> LED_SMD:LED_0805_2012Metric_Pad1.15x1.40mm_HandSolder
- J2, J5: footprint Connector_JST:JST_PH_S2B-PH-SM4-TB_1x02-1MP_P2.00mm_Horizontal -> Connector_PinHeader_2.54mm:PinHeader_1x02_P2.54mm_Vertical
- J4: symbol Connector:Micro_SD_Card -> Connector:Micro_SD_Card_Det
- R1, R11, R13, R14, R2, R3, R4, R6, R7, R8, R9: footprint Resistor_SMD:R_0402_1005Metric -> Resistor_SMD:R_0805_2012Metric_Pad1.15x1.40mm_HandSolder
Connections:
- net labels removed: IMU_INT
- wire segments 110 -> 106
- no-connect marks 25 -> 30
Changed lines of the file:
@@
 F 0 "C1" H 1315 4396 50  0000 L CNN
 F 1 "100n" H 1315 4305 50  0000 L CNN
-F 2 "Capacitor_SMD:C_0402_1005Metric" H 1238 4200 50  0001 C CNN
+F 2 "Capacitor_SMD:C_0805_2012Metric_Pad1.15x1.40mm_HandSolder" H 1238 4200 50  0001 C CNN
 F 3 "~" H 1200 4350 50  0001 C CNN
 	1    1200 4350
@@
 F 0 "C2" H 915 4396 50  0000 L CNN
 F 1 "2u2" H 915 4305 50  0000 L CNN
-F 2 "Capacitor_SMD:C_0402_1005Metric" H 838 4200 50  0001 C CNN
+F 2 "Capacitor_SMD:C_0805_2012Metric_Pad1.15x1.40mm_HandSolder" H 838 4200 50  0001 C CNN
 F 3 "~" H 800 4350 50  0001 C CNN
 	1    800  4350
@@
 $EndComp
 $Comp
-L Connector:Micro_SD_Card J4
+L Connector:Micro_SD_Card_Det J4
 U 1 1 5CB6F6D4
-P 9950 5650
-F 0 "J4" H 9900 6367 50  0000 C CNN
-F 1 "Micro_SD_Card" H 9900 6276 50  0000 C CNN
-F 2 "Connector_Card:microSD_HC_Hirose_DM3D-SF" H 11100 5950 50  0001 C CNN
-F 3 "http://katalog.we-online.de/em/datasheet/693072010801.pdf" H 9950 5650 50  0001 C CNN
-	1    9950 5650
+P 9950 5750
+F 0 "J4" H 9900 6467 50  0000 C CNN
+F 1 "Micro_SD_Card" H 9900 6376 50  0000 C CNN
+F 2 "Connector_Card:microSD_HC_Hirose_DM3D-SF" H 11100 6050 50  0001 C CNN
+F 3 "http://katalog.we-online.de/em/datasheet/693072010801.pdf" H 9950 5750 50  0001 C CNN
+	1    9950 5750
 	1    0    0    -1
 $EndComp
@@
 F 0 "C8" V 8421 1450 50  0000 C CNN
 F 1 "100n" V 8512 1450 50  0000 C CNN
-F 2 "Capacitor_SMD:C_0402_1005Metric" H 8650 1450 50  0001 C CNN
+F 2 "Capacitor_SMD:C_0805_2012Metric_Pad1.15x1.40mm_HandSolder" H 8650 1450 50  0001 C CNN
 F 3 "~" H 8650 1450 50  0001 C CNN
 	1    8650 1450
@@
 Text GLabel 4700 4550 0    50   Input ~ 0
 RXD0
-$Comp
-L power:+3V3 #PWR0105
-U 1 1 5CB86DE9
-P 4200 4650
-F 0 "#PWR0105" H 4200 4500 50  0001 C CNN
-F 1 "+3V3" V 4215 4778 50  0000 L CNN
-F 2 "" H 4200 4650 50  0001 C CNN
-F 3 "" H 4200 4650 50  0001 C CNN
-	1    4200 4650
-	0    -1   -1   0
-$EndComp
 Text GLabel 4700 4750 0    50   Input ~ 0
 IO0
@@
 F 0 "R1" H 870 2796 50  0000 L CNN
 F 1 "10K" H 870 2705 50  0000 L CNN
-F 2 "Resistor_SMD:R_0402_1005Metric" V 730 2750 50  0001 C CNN
+F 2 "Resistor_SMD:R_0805_2012Metric_Pad1.15x1.40mm_HandSolder" V 730 2750 50  0001 C CNN
 F 3 "~" H 800 2750 50  0001 C CNN
 	1    800  2750
@@
 F 0 "R4" H 1270 2796 50  0000 L CNN
 F 1 "10K" H 1270 2705 50  0000 L CNN
-F 2 "Resistor_SMD:R_0402_1005Metric" V 1130 2750 50  0001 C CNN
+F 2 "Resistor_SMD:R_0805_2012Metric_Pad1.15x1.40mm_HandSolder" V 1130 2750 50  0001 C CNN
 F 3 "~" H 1200 2750 50  0001 C CNN
 	1    1200 2750
@@
 F 0 "C3" H 3565 7196 50  0000 L CNN
 F 1 "47u" H 3565 7105 50  0000 L CNN
-F 2 "Capacitor_SMD:C_0805_2012Metric" H 3488 7000 50  0001 C CNN
+F 2 "Capacitor_SMD:C_0805_2012Metric_Pad1.15x1.40mm_HandSolder" H 3488 7000 50  0001 C CNN
 F 3 "~" H 3450 7150 50  0001 C CNN
 	1    3450 7150
@@
 F 0 "C4" H 4465 7196 50  0000 L CNN
 F 1 "47u" H 4465 7105 50  0000 L CNN
-F 2 "Capacitor_SMD:C_0805_2012Metric" H 4388 7000 50  0001 C CNN
+F 2 "Capacitor_SMD:C_0805_2012Metric_Pad1.15x1.40mm_HandSolder" H 4388 7000 50  0001 C CNN
 F 3 "~" H 4350 7150 50  0001 C CNN
 	1    4350 7150
@@
 Wire Wire Line
 	4350 7300 3900 7300
-$Comp
-L Device:C C6
-U 1 1 5CBBCFD7
-P 4750 7150
-F 0 "C6" H 4865 7196 50  0000 L CNN
-F 1 "nc" H 4865 7105 50  0000 L CNN
-F 2 "Capacitor_SMD:C_0402_1005Metric" H 4788 7000 50  0001 C CNN
-F 3 "~" H 4750 7150 50  0001 C CNN
-	1    4750 7150
-	1    0    0    -1
-$EndComp
-Wire Wire Line
-	4850 6950 4750 6950
 Connection ~ 4350 6950
-Wire Wire Line
-	4750 7000 4750 6950
-Connection ~ 4750 6950
-Wire Wire Line
-	4750 6950 4350 6950
-Wire Wire Line
-	4750 7300 4350 7300
-Connection ~ 4350 7300
 Text GLabel 8450 1950 0    50   Input ~ 0
 IMU_SCL
@@
 F 0 "C7" V 8500 6300 50  0000 L CNN
 F 1 "100n" V 8700 6250 50  0000 L CNN
-F 2 "Capacitor_SMD:C_0402_1005Metric" H 8600 6350 50  0001 C CNN
+F 2 "Capacitor_SMD:C_0805_2012Metric_Pad1.15x1.40mm_HandSolder" H 8600 6350 50  0001 C CNN
 F 3 "~" H 8600 6350 50  0001 C CNN
 	1    8600 6350
@@
 F 0 "R14" H 9000 5000 50  0000 L CNN
 F 1 "10K" H 9000 4900 50  0000 L CNN
-F 2 "Resistor_SMD:R_0402_1005Metric" H 8950 4950 50  0001 C CNN
+F 2 "Resistor_SMD:R_0805_2012Metric_Pad1.15x1.40mm_HandSolder" H 8950 4950 50  0001 C CNN
 F 3 "~" H 8950 4950 50  0001 C CNN
 	1    8950 4950
@@
 F 0 "R13" H 8900 4700 50  0000 L CNN
 F 1 "10K" H 8900 4600 50  0000 L CNN
-F 2 "Resistor_SMD:R_0402_1005Metric" H 8850 4650 50  0001 C CNN
+F 2 "Resistor_SMD:R_0805_2012Metric_Pad1.15x1.40mm_HandSolder" H 8850 4650 50  0001 C CNN
 F 3 "~" H 8850 4650 50  0001 C CNN
 	1    8850 4650
@@
 F 0 "R7" H 8450 5000 50  0000 L CNN
 F 1 "10K" H 8450 4900 50  0000 L CNN
-F 2 "Resistor_SMD:R_0402_1005Metric" H 8400 4950 50  0001 C CNN
+F 2 "Resistor_SMD:R_0805_2012Metric_Pad1.15x1.40mm_HandSolder" H 8400 4950 50  0001 C CNN
 F 3 "~" H 8400 4950 50  0001 C CNN
 	1    8400 4950
@@
 F 0 "R9" H 8600 4700 50  0000 L CNN
 F 1 "10K" H 8600 4600 50  0000 L CNN
-F 2 "Resistor_SMD:R_0402_1005Metric" H 8550 4650 50  0001 C CNN
+F 2 "Resistor_SMD:R_0805_2012Metric_Pad1.15x1.40mm_HandSolder" H 8550 4650 50  0001 C CNN
 F 3 "~" H 8550 4650 50  0001 C CNN
 	1    8550 4650
@@
 F 0 "R11" H 8700 5000 50  0000 L CNN
 F 1 "10K" H 8700 4900 50  0000 L CNN
-F 2 "Resistor_SMD:R_0402_1005Metric" H 8650 4950 50  0001 C CNN
+F 2 "Resistor_SMD:R_0805_2012Metric_Pad1.15x1.40mm_HandSolder" H 8650 4950 50  0001 C CNN
 F 3 "~" H 8650 4950 50  0001 C CNN
 	1    8650 4950
@@
 Text GLabel 2800 3250 2    50   Input ~ 0
 IMU_SCL
-Text GLabel 10500 2050 2    50   Input ~ 0
-IMU_INT
-$Comp
-L Device:R_Small R17
-U 1 1 5CC9A8BF
-P 10000 2050
-F 0 "R17" V 10050 2050 50  0000 C CNN
-F 1 "nc" V 9950 2050 50  0000 C CNN
-F 2 "Resistor_SMD:R_0402_1005Metric" H 10000 2050 50  0001 C CNN
-F 3 "~" H 10000 2050 50  0001 C CNN
-	1    10000 2050
-	0    -1   -1   0
-$EndComp
-Wire Wire Line
-	10100 2050 10500 2050
 Wire Wire Line
 	8900 1650 8750 1650
@@
 Wire Wire Line
 	8550 1750 8900 1750
-Text GLabel 2800 3350 2    50   Input ~ 0
-IMU_INT
-$Comp
-L Device:R_Small R5
-U 1 1 5CCD8A95
-P 4300 4650
-F 0 "R5" V 4350 4650 50  0000 C CNN
-F 1 "nc" V 4250 4650 50  0000 C CNN
-F 2 "Resistor_SMD:R_0402_1005Metric" H 4300 4650 50  0001 C CNN
-F 3 "~" H 4300 4650 50  0001 C CNN
-	1    4300 4650
-	0    -1   -1   0
-$EndComp
-Wire Wire Line
-	4700 4650 4400 4650
 Wire Wire Line
 	8450 1950 8900 1950
@@
 F 0 "R2" H 8200 5000 50  0000 L CNN
 F 1 "nc" H 8200 4900 50  0000 L CNN
-F 2 "Resistor_SMD:R_0402_1005Metric" H 8150 4950 50  0001 C CNN
+F 2 "Resistor_SMD:R_0805_2012Metric_Pad1.15x1.40mm_HandSolder" H 8150 4950 50  0001 C CNN
 F 3 "~" H 8150 4950 50  0001 C CNN
 	1    8150 4950
@@
 F 0 "C9" H 4592 1946 50  0000 L CNN
 F 1 "4.7u" H 4592 1855 50  0000 L CNN
-F 2 "Capacitor_SMD:C_0402_1005Metric" H 4500 1900 50  0001 C CNN
+F 2 "Capacitor_SMD:C_0805_2012Metric_Pad1.15x1.40mm_HandSolder" H 4500 1900 50  0001 C CNN
 F 3 "~" H 4500 1900 50  0001 C CNN
 	1    4500 1900
@@
 F 0 "C10" H 6142 1896 50  0000 L CNN
 F 1 "4.7u" H 6142 1805 50  0000 L CNN
-F 2 "Capacitor_SMD:C_0402_1005Metric" H 6050 1850 50  0001 C CNN
+F 2 "Capacitor_SMD:C_0805_2012Metric_Pad1.15x1.40mm_HandSolder" H 6050 1850 50  0001 C CNN
 F 3 "~" H 6050 1850 50  0001 C CNN
 	1    6050 1850
@@
 F 0 "R3" H 5009 2196 50  0000 L CNN
 F 1 "2k" H 5009 2105 50  0000 L CNN
-F 2 "Resistor_SMD:R_0402_1005Metric" H 4950 2150 50  0001 C CNN
+F 2 "Resistor_SMD:R_0805_2012Metric_Pad1.15x1.40mm_HandSolder" H 4950 2150 50  0001 C CNN
 F 3 "~" H 4950 2150 50  0001 C CNN
 	1    4950 2150
@@
 F 0 "D2" V 6689 1783 50  0000 R CNN
 F 1 "LED" V 6598 1783 50  0000 R CNN
-F 2 "LED_SMD:LED_0402_1005Metric" H 6650 1900 50  0001 C CNN
+F 2 "LED_SMD:LED_0805_2012Metric_Pad1.15x1.40mm_HandSolder" H 6650 1900 50  0001 C CNN
 F 3 "~" H 6650 1900 50  0001 C CNN
 	1    6650 1900
@@
 F 0 "R6" V 6354 2050 50  0000 C CNN
 F 1 "470" V 6445 2050 50  0000 C CNN
-F 2 "Resistor_SMD:R_0402_1005Metric" H 6550 2050 50  0001 C CNN
+F 2 "Resistor_SMD:R_0805_2012Metric_Pad1.15x1.40mm_HandSolder" H 6550 2050 50  0001 C CNN
 F 3 "~" H 6550 2050 50  0001 C CNN
 	1    6550 2050
@@
 F 0 "J2" H 4580 2692 50  0000 L CNN
 F 1 "BATCONN" H 4580 2601 50  0000 L CNN
-F 2 "Connector_JST:JST_PH_S2B-PH-SM4-TB_1x02-1MP_P2.00mm_Horizontal" H 4500 2700 50  0001 C CNN
+F 2 "Connector_PinHeader_2.54mm:PinHeader_1x02_P2.54mm_Vertical" H 4500 2700 50  0001 C CNN
 F 3 "~" H 4500 2700 50  0001 C CNN
 	1    4500 2700
@@
 F 0 "R8" H 1709 7196 50  0000 L CNN
 F 1 "10k" H 1709 7105 50  0000 L CNN
-F 2 "Resistor_SMD:R_0402_1005Metric" H 1650 7150 50  0001 C CNN
+F 2 "Resistor_SMD:R_0805_2012Metric_Pad1.15x1.40mm_HandSolder" H 1650 7150 50  0001 C CNN
 F 3 "~" H 1650 7150 50  0001 C CNN
 	1    1650 7150
@@
 $EndComp
 Wire Wire Line
-	1950 6900 1650 6900
+	1950 6900 1850 6900
 Wire Wire Line
 	1650 6900 1650 7050
@@
 F 0 "J5" H 1080 6992 50  0000 L CNN
 F 1 "PWRCONN" H 1080 6901 50  0000 L CNN
-F 2 "Connector_JST:JST_PH_S2B-PH-SM4-TB_1x02-1MP_P2.00mm_Horizontal" H 1000 7000 50  0001 C CNN
+F 2 "Connector_PinHeader_2.54mm:PinHeader_1x02_P2.54mm_Vertical" H 1000 7000 50  0001 C CNN
 F 3 "~" H 1000 7000 50  0001 C CNN
 	1    1000 7000
@@
 	1    0    0    -1
 $EndComp
+$Comp
+L power:PWR_FLAG #FLG0104
+U 1 1 5CBCC836
+P 1850 6900
+F 0 "#FLG0104" H 1850 6975 50  0001 C CNN
+F 1 "PWR_FLAG" H 1850 7073 50  0000 C CNN
+F 2 "" H 1850 6900 50  0001 C CNN
+F 3 "~" H 1850 6900 50  0001 C CNN
+	1    1850 6900
+	1    0    0    -1
+$EndComp
+Connection ~ 1850 6900
+Wire Wire Line
+	1850 6900 1650 6900
+NoConn ~ 4700 4650
+Wire Wire Line
+	4350 6950 4850 6950
+NoConn ~ 9900 2050
+NoConn ~ 2800 3350
+NoConn ~ 9050 6150
+NoConn ~ 9050 6250
 $EndSCHEMATC
