File: imulogger/imulogger.kicad_pcb (KiCad board)
At the start: 2 copper layers, 64 x 25 mm, 31 parts, among them J1 DEBUG, J2 BATCONN, J4 Micro_SD_Card, J5 PWRCONN, Q1 TP0610T, U1 ESP32-WROOM-32, U2 USFS, U3 MCP1826S, U4 MCP73831-2-OT

Commit message: pcb optimizations
Parts:
- moved C8 20.5 mm to (167.4, 77.3)
- moved C2 10.4 mm to (123.0, 76.0), turned to 0 degrees
- moved J2 0.50 mm to (162.0, 80.5)
- turned U2 to 0 degrees
Routing:
- net IMU_SDA: track 62.2 -> 37.8 mm
- net +3V3: track 133.2 -> 112.9 mm
- net IMU_SCL: track 65.1 -> 48.9 mm
- net GND: track 63.5 -> 70.1 mm, vias 44 -> 67
- net EN: track 27.4 -> 25.3 mm
